File: CutSheetSensors.kicad_sch (KiCad schematic)
At the start: 3 parts, among them J1 Conn_01x03_MountingPin, J2 Conn_01x03_MountingPin, J3 Conn_01x03_MountingPin

Commit message: 10/09/23 - Schematic v0.1
Parts:
- J1, J2, J3: value Conn_01x03_MountingPin -> JST PH S3B
Connections:
- net EDGE_DETECTOR: now reaches J2.2 (Pin_2)
- net PHOTO_EYE_LEFT: now reaches J1.2 (Pin_2)
- net PHOTO_EYE_RIGHT: now reaches J3.2 (Pin_2)
Other:
- moved on the sheet: J1, J2, J3
