File: IndicatorLEDs.kicad_sch (KiCad schematic)
At the start: 7 parts, among them J6 Conn_01x05_MountingPin, Q4 NMOS, Q5 NMOS, Q6 NMOS

Commit message: 10/09/23 - Schematic v0.1
Parts:
- added R10 (x3): 100k, Resistor_SMD:R_0402_1005Metric, symbol Device:R_Small_US
Connections:
- net GND: now also R10.2, R10.2, R10.2
- net LED_CTRL_1: now also R10.1
- net LED_CTRL_2: now also R10.1
- net LED_CTRL_3: now also R10.1
Other:
- moved on the sheet: J6, Q4, Q6, R5, R7
