File: Motors_Encoders.kicad_sch (KiCad schematic)
At the start: 17 parts, among them J4 Conn_01x06_MountingPin, J5 Conn_01x12_MountingPin, Q1 NMOS, Q2 NMOS, Q3 NMOS, U1 DRV8847RTE, U2 DRV8847RTE

Commit message: 10/09/23 - Schematic v0.1
Parts:
- added R10, R11, R12: 100k, Resistor_SMD:R_0402_1005Metric, symbol Device:R_Small_US
- NT1, NT2: footprint (none) -> NetTie:NetTie-2_SMD_Pad0.5mm
Connections:
- net ENC_CTRL_1: now also R10.1
- net ENC_CTRL_2: now also R12.1
- net ENC_CTRL_3: now also R11.1
- net GND: now also R10.2, R11.2, R12.2
- net MODE_1: now reaches U2.12 (MODE)
- net IN2_1: now reaches U2.13 (IN2)
- net IN1_1: now reaches U2.14 (IN1)
- net ~{SLEEP}_1: now reaches U2.15 (~{SLEEP})
- net ~{FAULT}_1: now reaches U2.6 (~{FAULT})
- net TRQ_1: now reaches U2.9 (TRQ)
- net MODE_2/3: now reaches U1.12 (MODE)
- net IN2_2/3: now reaches U1.13 (IN2)
- net IN1_2/3: now reaches U1.14 (IN1)
- net ~{SLEEP}_2/3: now reaches U1.15 (~{SLEEP})
- net ~{FAULT}_2/3: now reaches U1.6 (~{FAULT})
- net IN3_2/3: now reaches U1.7 (IN3)
- net IN4_2/3: now reaches U1.8 (IN4)
- net TRQ_2/3: now reaches U1.9 (TRQ)
- no-connect marks 2 -> 4
Other:
- moved on the sheet: Q2, Q3
